File: Headphone Amps/CMoy-Pro/SMD-No_Pot/CMoy-Pro-Buffer-Board-V_1_0_0_1a.sch (EAGLE design)
At the start: 24 parts

Commit message: Changes from surface book
These are the files that have changed on the surface book. I have not tracked the project individually.
Parts:
- R1, R2: device common:RES0805L3 -> common:RES1210L3
