File: Headphone Amps/CMoy-Pro/SMD-No_Pot/CMoy-Pro-Buffer-Board-V_1_0_0_1a.brd (EAGLE design)
At the start: 28.9 x 28.9 mm, 24 parts

Commit message: Changes from surface book
These are the files that have changed on the surface book. I have not tracked the project individually.
Parts:
- R1, R2: device common:0805L3 -> common:1210L3
- moved JP2 5.08 mm to (26.4, 17.3)
- moved R2 0.84 mm to (21.1, 11.4)
- moved R1 0.84 mm to (21.1, 17.5)
- moved L1 0.20 mm to (21.1, 19.9)
- moved L2 0.20 mm to (21.1, 8.94)
- flipped C1 to the bottom
- flipped C2 to the bottom
- flipped C3 to the bottom
- flipped C4 to the bottom
Connections:
- net N$1: now also R2.P$1; no longer R2.1
- net N$2: now also R2.P$2; no longer R2.2
- net N$4: now also R1.P$1; no longer R1.1
- net N$5: now also R1.P$2; no longer R1.2
Routing:
- net N$1: track 18.1 -> 5.10 mm
- net N$4: track 18.1 -> 5.10 mm
- net N$5: track 12.2 -> 0.05 mm
- net N$2: track 10.3 -> 0.02 mm
- net N$12: track 25.3 -> 20.3 mm
- added copper zone on layer 1, net N$1
- added copper zone on layer 1, net N$2
- added copper zone on layer 1, net N$4
- removed copper zone on layer 1, net GND
- removed copper zone on layer 16, net GND
- removed copper zone on layer 16, net V+
- removed copper zone on layer 16, net V-

Commit message: Several Projects
Projects - Vape - USB Microphone - USB Hub - Headphone Amps - Backpack
Parts:
- moved C7 0.61 mm to (5.89, 22.4), turned to 225 degrees
- moved C8 0.61 mm to (5.89, 6.50), turned to 315 degrees
- moved R1 0.20 mm to (21.3, 17.5)
- moved R2 0.20 mm to (21.3, 11.4)
- turned C1 to 180 degrees
- turned C3 to 180 degrees
- flipped C5 to the bottom
- flipped C6 to the bottom
Routing:
- net N$4: track 5.10 -> 12.2 mm
- net N$1: track 5.10 -> 12.2 mm
- net N$8: track 20.5 -> 19.4 mm
- added copper zone on layer 1, net N$5
- added copper zone on layer 16, net V+
- added copper zone on layer 16, net V-
