File: BackPack/backpack_board.sch (EAGLE design)
At the start: 9 parts, among them IC1 LT1963EST-3.3, X1 SATA7-32009-10X

Commit message: Several Projects
Projects - Vape - USB Microphone - USB Hub - Headphone Amps - Backpack
Parts:
- removed X1: SATA7-32009-10X, con-cypressindustries:SATA7-32009-10X
- added X2: SATA7-32009-10X, con-cypressindustries:SATA7-32009-10X
Connections:
- net 1_N renamed USB0_SSTX_N
- net 1_P renamed USB0_SSTX_P
- net 2_N renamed USB0_SSRX_N
- net 2_P renamed USB0_SSRX_P
- net 3_N renamed USB0_HS_N
- net 3_P renamed USB0_HS_P
- net N$101: no longer X1.3
- net N$102: no longer X1.1
- net N$103: no longer X1.7
- net N$104: no longer X1.5
