File: USB Hub/4-Port/tusb8041_hub_test.brd (EAGLE design)
At the start: 64.5 x 64 mm, 116 parts

Commit message: Several Projects
Projects - Vape - USB Microphone - USB Hub - Headphone Amps - Backpack
Parts:
- added R19, R20: 4.7K, common:0402L3
- CN2: value (none) -> BRD_5V
- LED1: value (none) -> VBUS1
- LED2: value (none) -> VBUS2
- LED3: value (none) -> VBUS3
- LED4: value (none) -> VBUS4
- LED5: value (none) -> PWR
- LED6: value (none) -> SS_UP
- LED7: value (none) -> HS_UP
- R10, R16, R18, R6, R8, R9: value (none) -> 220R
- U1: value (none) -> USB_HUB
- U2, U3, U4, U5: value (none) -> USB_5V
- U6: value (none) -> BRD_3V3
- U8: value (none) -> BRD_1V1
- moved C68 0.13 mm to (141.1, 75.6)
Connections:
- net PWRCTL3: now also R20.P$2, U1.33
- net PWRCTL4: now also R19.P$2, U1.32
- net VDD33: now also R19.P$1, R20.P$1
Routing:
- net PWRCTL4: track 5.55 -> 8.86 mm
- net VDD33: track 13.7 -> 15.7 mm, vias 13 -> 15
- net CLK_P: track 12.6 -> 11.3 mm
